Commit message: 修改：     robot_control/launch/sim_with_py_controller.launch 	修改：     robot_control/scripts/imu_do_node.py 	修改：     robot_control/scripts/k_update.py 	修改：     robot_control/scripts/lqr_control.py 	修改：     robot_control/scripts/lqr_control1.py 	修改：     robot_control/scripts/multi_receive.py 	修改：     robot_control/scripts/online_lqr.py 	修改：     robot_control/scripts/online_lqr1.py 	修改：     robot_description/launch/gazebo_sim.launch 	修改：     robot_description/launch/my_world.launch 	修改：     robot_description/urdf/wbrobot.urdf

File: robot_description/urdf/wbrobot.urdf (robot description, URDF)
Before this commit: robot wbrobot, 8 links, 7 joints
Joints:
- joint datui1_joint: origin xyz=-0.08 0 0 rpy=-3.1416 0 3.1416 -> xyz=-0.08 0 0 rpy=2.923 0 3.1416
- joint datui2_joint: origin xyz=0.08 0 0 rpy=0 0 0 -> xyz=0.08 0 0 rpy=0.218 0 0

Commit message: old urdf

File: robot_description/urdf/wbrobot.urdf (robot description, URDF)
Before this commit: robot wbrobot, 8 links, 7 joints
Links:
- added link hokuyo_link, mass 0; collision box size=0.1 0.1 0.1; visual cylinder length=0.1 radius=0.04
Joints:
- added joint hokuyo_joint: type fixed, parent base_link, child hokuyo_link, origin xyz=0 0 0.1 rpy=0 0 0, axis 0 1 0

Commit message: 可以建图但是里程计不行

File: robot_description/urdf/wbrobot.urdf (robot description, URDF)
Before this commit: robot wbrobot, 9 links, 8 joints
Joints:
- joint hokuyo_joint: origin xyz=0 0 0.1 rpy=0 0 0 -> xyz=0 0 0.1 rpy=0 0 1.57

Commit message: mapping done

File: robot_description/urdf/wbrobot.urdf (robot description, URDF)
Before this commit: robot wbrobot, 9 links, 8 joints
Links:
- added link base_footprint
Joints:
- added joint footprint: type fixed, parent base_footprint, child base_link, origin xyz=0 0 0.21 rpy=0 0 -1.57
- joint world_joint: child base_link -> base_footprint; origin xyz=0 0 0.13 rpy=0 0 0 -> xyz=0.0 0.0 0.0 rpy=0.0 0.0 1.57
